Commit message: configurig localizers motion model

File: src/husky-kinetic-devel/husky_description/urdf/accessories/sick_lms1xx_mount.urdf.xacro (robot description, xacro)
@@ -45,5 +45,5 @@
     <joint name="${prefix}_laser_joint" type="fixed">
       <!-- This offset is from the base of the bracket to the LIDAR's focal point. -->
-      <origin xyz="0.0352 0 0.0566" rpy="0 0 0" /> <!-- ${M_PI} 0 0, this sets the laser with z-axis pointing downwards--> <!-- 0 0 0, this sets the laser with z-axis pointing upwards-->
+      <origin xyz="0.0352 0 0.0566" rpy="${M_PI} 0 0" /> <!-- ${M_PI} 0 0, this sets the laser with z-axis pointing downwards, good for gmapping--> <!-- 0 0 0, this sets the laser with z-axis pointing upwards-->
       <parent link="${prefix}_laser_mount" />
       <child link="${prefix}_laser" />

File: src/husky-kinetic-devel/husky_description/urdf/husky.urdf.xacro (robot description, xacro)
@@ -22,5 +22,5 @@
 -->
 <robot name="husky" xmlns:xacro="http://ros.org/wiki/xacro">
-  <xacro:arg name="laser_enabled" default="true" />
+  <xacro:arg name="laser_enabled" default="false" />
   <xacro:arg name="laser_xyz" default="$(optenv HUSKY_LMS1XX_XYZ 0.2206 0.0 0.00635)" />
   <xacro:arg name="laser_rpy" default="$(optenv HUSKY_LMS1XX_RPY 0.0 0.0 0.0)" />

File: src/husky-kinetic-devel/husky_description/urdf/sick_lms1xx.urdf.xacro (robot description, xacro)
@@ -28,5 +28,5 @@
 <robot xmlns:xacro="http://ros.org/wiki/xacro">
   <xacro:macro name="sick_lms1xx" params="frame:=laser topic:=scan sample_size:=720 update_rate:=50
-               min_angle:=-3.1415 max_angle:=3.1415 min_range:=0.3 max_range:=60.0 robot_namespace:=/" >
+               min_angle:=-3.1415 max_angle:=3.1415 min_range:=0.3 max_range:=30.0 robot_namespace:=/" >
     <link name="${frame}">
       <inertial>
